File: Hardware/Chebyshev_Input_BPF_R0.sch (KiCad schematic (older format))
At the start: 9 parts

Commit message: Major cleanup to both the schematic and directory structure. Stackup has changed accomodate to 0.65mm trace width. Chebyshev filter lived through the experience in the Qucs simulation; others not checked yet. I do want to re-visit the matching networks of all of the amplifiers as I have developed some good strategies to implement them.
Parts:
- renumbered C45 to C16, C46 to C17, C47 to C18, C48 to C19, C49 to C20, C50 to C21, L19 to L6, L20 to L7, L21 to L8
Changed lines of the file:
@@
 $Descr A4 11693 8268
 encoding utf-8
-Sheet 16 16
+Sheet 22 24
 Title ""
 Date ""
@@
 P 3400 3950
 AR Path="/5F177657/5F1A3D70" Ref="C?"  Part="1"
-AR Path="/5F20B396/5F216BC6/5F1A3D70" Ref="C45"  Part="1"
-F 0 "C45" H 3515 3996 50  0000 L CNN
+AR Path="/5F20B396/5F216BC6/5F1A3D70" Ref="C16"  Part="1"
+F 0 "C16" H 3515 3996 50  0000 L CNN
 F 1 "600S100" H 3515 3905 50  0000 L CNN
 F 2 "Capacitor_SMD:C_0603_1608Metric" H 3450 4050 50  0001 C CNN
@@
 P 5000 3950
 AR Path="/5F177657/5F1A44C9" Ref="C?"  Part="1"
-AR Path="/5F20B396/5F216BC6/5F1A44C9" Ref="C46"  Part="1"
-F 0 "C46" H 5115 3996 50  0000 L CNN
+AR Path="/5F20B396/5F216BC6/5F1A44C9" Ref="C17"  Part="1"
+F 0 "C17" H 5115 3996 50  0000 L CNN
 F 1 "600S220" H 5115 3905 50  0000 L CNN
 F 2 "Capacitor_SMD:C_0603_1608Metric" H 5050 4050 50  0001 C CNN
@@
 P 5350 3600
 AR Path="/5F177657/5F1A4BFC" Ref="C?"  Part="1"
-AR Path="/5F20B396/5F216BC6/5F1A4BFC" Ref="C47"  Part="1"
-F 0 "C47" V 5098 3600 50  0000 C CNN
+AR Path="/5F20B396/5F216BC6/5F1A4BFC" Ref="C18"  Part="1"
+F 0 "C18" V 5098 3600 50  0000 C CNN
 F 1 "600S2R7" V 5189 3600 50  0000 C CNN
 F 2 "Capacitor_SMD:C_0603_1608Metric" H 5400 3700 50  0001 C CNN
@@
 P 5950 3600
 AR Path="/5F177657/5F1A551B" Ref="L?"  Part="1"
-AR Path="/5F20B396/5F216BC6/5F1A551B" Ref="L20"  Part="1"
-F 0 "L20" H 5950 3815 50  0000 C CNN
+AR Path="/5F20B396/5F216BC6/5F1A551B" Ref="L7"  Part="1"
+F 0 "L7" H 5950 3815 50  0000 C CNN
 F 1 "0603HP-82NX" H 5950 3724 50  0000 C CNN
 F 2 "Inductor_SMD:L_0603_1608Metric" H 5700 3750 50  0001 C CNN
@@
 P 8500 3950
 AR Path="/5F177657/5F1AC139" Ref="C?"  Part="1"
-AR Path="/5F20B396/5F216BC6/5F1AC139" Ref="C50"  Part="1"
-F 0 "C50" H 8615 3996 50  0000 L CNN
+AR Path="/5F20B396/5F216BC6/5F1AC139" Ref="C21"  Part="1"
+F 0 "C21" H 8615 3996 50  0000 L CNN
 F 1 "600S100" H 8615 3905 50  0000 L CNN
 F 2 "Capacitor_SMD:C_0603_1608Metric" H 8550 4050 50  0001 C CNN
@@
 P 6900 3950
 AR Path="/5F177657/5F1AC13F" Ref="C?"  Part="1"
-AR Path="/5F20B396/5F216BC6/5F1AC13F" Ref="C49"  Part="1"
-F 0 "C49" H 6785 3904 50  0000 R CNN
+AR Path="/5F20B396/5F216BC6/5F1AC13F" Ref="C20"  Part="1"
+F 0 "C20" H 6785 3904 50  0000 R CNN
 F 1 "600S220" H 6785 3995 50  0000 R CNN
 F 2 "Capacitor_SMD:C_0603_1608Metric" H 6950 4050 50  0001 C CNN
@@
 P 7700 4050
 AR Path="/5F177657/5F1AC145" Ref="L?"  Part="1"
-AR Path="/5F20B396/5F216BC6/5F1AC145" Ref="L21"  Part="1"
-F 0 "L21" V 7746 4127 50  0000 L CNN
+AR Path="/5F20B396/5F216BC6/5F1AC145" Ref="L8"  Part="1"
+F 0 "L8" V 7746 4127 50  0000 L CNN
 F 1 "0603HP-3N6X" V 7655 4127 50  0000 L CNN
 F 2 "Inductor_SMD:L_0603_1608Metric" H 7450 4200 50  0001 C CNN
@@
 P 6550 3600
 AR Path="/5F177657/5F1AC14B" Ref="C?"  Part="1"
-AR Path="/5F20B396/5F216BC6/5F1AC14B" Ref="C48"  Part="1"
-F 0 "C48" V 6298 3600 50  0000 C CNN
+AR Path="/5F20B396/5F216BC6/5F1AC14B" Ref="C19"  Part="1"
+F 0 "C19" V 6298 3600 50  0000 C CNN
 F 1 "600S2R7" V 6389 3600 50  0000 C CNN
 F 2 "Capacitor_SMD:C_0603_1608Metric" H 6600 3700 50  0001 C CNN
@@
 P 4200 4050
 AR Path="/5F177657/5F1BFC4F" Ref="L?"  Part="1"
-AR Path="/5F20B396/5F216BC6/5F1BFC4F" Ref="L19"  Part="1"
-F 0 "L19" V 4246 4127 50  0000 L CNN
+AR Path="/5F20B396/5F216BC6/5F1BFC4F" Ref="L6"  Part="1"
+F 0 "L6" V 4246 4127 50  0000 L CNN
 F 1 "0603HP-3N6X" V 4155 4127 50  0000 L CNN
 F 2 "Inductor_SMD:L_0603_1608Metric" H 3950 4200 50  0001 C CNN
@@
 P 3400 4300
 AR Path="/5F177657/5F1DD62C" Ref="#PWR?"  Part="1"
-AR Path="/5F20B396/5F216BC6/5F1DD62C" Ref="#PWR057"  Part="1"
-F 0 "#PWR057" H 3400 4050 50  0001 C CNN
+AR Path="/5F20B396/5F216BC6/5F1DD62C" Ref="#PWR023"  Part="1"
+F 0 "#PWR023" H 3400 4050 50  0001 C CNN
 F 1 "GNDA" H 3405 4127 50  0000 C CNN
 F 2 "" H 3400 4300 50  0001 C CNN
@@
 P 5000 4300
 AR Path="/5F177657/5F1DEE33" Ref="#PWR?"  Part="1"
-AR Path="/5F20B396/5F216BC6/5F1DEE33" Ref="#PWR059"  Part="1"
-F 0 "#PWR059" H 5000 4050 50  0001 C CNN
+AR Path="/5F20B396/5F216BC6/5F1DEE33" Ref="#PWR025"  Part="1"
+F 0 "#PWR025" H 5000 4050 50  0001 C CNN
 F 1 "GNDA" H 5005 4127 50  0000 C CNN
 F 2 "" H 5000 4300 50  0001 C CNN
@@
 P 4200 4500
 AR Path="/5F177657/5F1DF153" Ref="#PWR?"  Part="1"
-AR Path="/5F20B396/5F216BC6/5F1DF153" Ref="#PWR058"  Part="1"
-F 0 "#PWR058" H 4200 4250 50  0001 C CNN
+AR Path="/5F20B396/5F216BC6/5F1DF153" Ref="#PWR024"  Part="1"
+F 0 "#PWR024" H 4200 4250 50  0001 C CNN
 F 1 "GNDA" H 4205 4327 50  0000 C CNN
 F 2 "" H 4200 4500 50  0001 C CNN
@@
 P 7700 4500
 AR Path="/5F177657/5F1E005D" Ref="#PWR?"  Part="1"
-AR Path="/5F20B396/5F216BC6/5F1E005D" Ref="#PWR061"  Part="1"
-F 0 "#PWR061" H 7700 4250 50  0001 C CNN
+AR Path="/5F20B396/5F216BC6/5F1E005D" Ref="#PWR027"  Part="1"
+F 0 "#PWR027" H 7700 4250 50  0001 C CNN
 F 1 "GNDA" H 7705 4327 50  0000 C CNN
 F 2 "" H 7700 4500 50  0001 C CNN
@@
 P 6900 4300
 AR Path="/5F177657/5F1E0461" Ref="#PWR?"  Part="1"
-AR Path="/5F20B396/5F216BC6/5F1E0461" Ref="#PWR060"  Part="1"
-F 0 "#PWR060" H 6900 4050 50  0001 C CNN
+AR Path="/5F20B396/5F216BC6/5F1E0461" Ref="#PWR026"  Part="1"
+F 0 "#PWR026" H 6900 4050 50  0001 C CNN
 F 1 "GNDA" H 6905 4127 50  0000 C CNN
 F 2 "" H 6900 4300 50  0001 C CNN
@@
 P 8500 4300
 AR Path="/5F177657/5F1E096E" Ref="#PWR?"  Part="1"
-AR Path="/5F20B396/5F216BC6/5F1E096E" Ref="#PWR062"  Part="1"
-F 0 "#PWR062" H 8500 4050 50  0001 C CNN
+AR Path="/5F20B396/5F216BC6/5F1E096E" Ref="#PWR028"  Part="1"
+F 0 "#PWR028" H 8500 4050 50  0001 C CNN
 F 1 "GNDA" H 8505 4127 50  0000 C CNN
 F 2 "" H 8500 4300 50  0001 C CNN

Commit message: Improving LNA simulations and Documentation package. More to come on this one.
Parts:
- renumbered C16 to C19, C17 to C20, C18 to C21, C19 to C22, C20 to C23, C21 to C24, L6 to L7, L7 to L8, L8 to L9
Changed lines of the file:
@@
 $Descr A4 11693 8268
 encoding utf-8
-Sheet 22 24
+Sheet 22 23
 Title ""
 Date ""
@@
 P 3400 3950
 AR Path="/5F177657/5F1A3D70" Ref="C?"  Part="1"
-AR Path="/5F20B396/5F216BC6/5F1A3D70" Ref="C16"  Part="1"
-F 0 "C16" H 3515 3996 50  0000 L CNN
+AR Path="/5F20B396/5F216BC6/5F1A3D70" Ref="C19"  Part="1"
+F 0 "C19" H 3515 3996 50  0000 L CNN
 F 1 "600S100" H 3515 3905 50  0000 L CNN
 F 2 "Capacitor_SMD:C_0603_1608Metric" H 3450 4050 50  0001 C CNN
@@
 P 5000 3950
 AR Path="/5F177657/5F1A44C9" Ref="C?"  Part="1"
-AR Path="/5F20B396/5F216BC6/5F1A44C9" Ref="C17"  Part="1"
-F 0 "C17" H 5115 3996 50  0000 L CNN
+AR Path="/5F20B396/5F216BC6/5F1A44C9" Ref="C20"  Part="1"
+F 0 "C20" H 5115 3996 50  0000 L CNN
 F 1 "600S220" H 5115 3905 50  0000 L CNN
 F 2 "Capacitor_SMD:C_0603_1608Metric" H 5050 4050 50  0001 C CNN
@@
 P 5350 3600
 AR Path="/5F177657/5F1A4BFC" Ref="C?"  Part="1"
-AR Path="/5F20B396/5F216BC6/5F1A4BFC" Ref="C18"  Part="1"
-F 0 "C18" V 5098 3600 50  0000 C CNN
+AR Path="/5F20B396/5F216BC6/5F1A4BFC" Ref="C21"  Part="1"
+F 0 "C21" V 5098 3600 50  0000 C CNN
 F 1 "600S2R7" V 5189 3600 50  0000 C CNN
 F 2 "Capacitor_SMD:C_0603_1608Metric" H 5400 3700 50  0001 C CNN
@@
 P 5950 3600
 AR Path="/5F177657/5F1A551B" Ref="L?"  Part="1"
-AR Path="/5F20B396/5F216BC6/5F1A551B" Ref="L7"  Part="1"
-F 0 "L7" H 5950 3815 50  0000 C CNN
+AR Path="/5F20B396/5F216BC6/5F1A551B" Ref="L8"  Part="1"
+F 0 "L8" H 5950 3815 50  0000 C CNN
 F 1 "0603HP-82NX" H 5950 3724 50  0000 C CNN
 F 2 "Inductor_SMD:L_0603_1608Metric" H 5700 3750 50  0001 C CNN
@@
 P 8500 3950
 AR Path="/5F177657/5F1AC139" Ref="C?"  Part="1"
-AR Path="/5F20B396/5F216BC6/5F1AC139" Ref="C21"  Part="1"
-F 0 "C21" H 8615 3996 50  0000 L CNN
+AR Path="/5F20B396/5F216BC6/5F1AC139" Ref="C24"  Part="1"
+F 0 "C24" H 8615 3996 50  0000 L CNN
 F 1 "600S100" H 8615 3905 50  0000 L CNN
 F 2 "Capacitor_SMD:C_0603_1608Metric" H 8550 4050 50  0001 C CNN
@@
 P 6900 3950
 AR Path="/5F177657/5F1AC13F" Ref="C?"  Part="1"
-AR Path="/5F20B396/5F216BC6/5F1AC13F" Ref="C20"  Part="1"
-F 0 "C20" H 6785 3904 50  0000 R CNN
+AR Path="/5F20B396/5F216BC6/5F1AC13F" Ref="C23"  Part="1"
+F 0 "C23" H 6785 3904 50  0000 R CNN
 F 1 "600S220" H 6785 3995 50  0000 R CNN
 F 2 "Capacitor_SMD:C_0603_1608Metric" H 6950 4050 50  0001 C CNN
@@
 P 7700 4050
 AR Path="/5F177657/5F1AC145" Ref="L?"  Part="1"
-AR Path="/5F20B396/5F216BC6/5F1AC145" Ref="L8"  Part="1"
-F 0 "L8" V 7746 4127 50  0000 L CNN
+AR Path="/5F20B396/5F216BC6/5F1AC145" Ref="L9"  Part="1"
+F 0 "L9" V 7746 4127 50  0000 L CNN
 F 1 "0603HP-3N6X" V 7655 4127 50  0000 L CNN
 F 2 "Inductor_SMD:L_0603_1608Metric" H 7450 4200 50  0001 C CNN
@@
 P 6550 3600
 AR Path="/5F177657/5F1AC14B" Ref="C?"  Part="1"
-AR Path="/5F20B396/5F216BC6/5F1AC14B" Ref="C19"  Part="1"
-F 0 "C19" V 6298 3600 50  0000 C CNN
+AR Path="/5F20B396/5F216BC6/5F1AC14B" Ref="C22"  Part="1"
+F 0 "C22" V 6298 3600 50  0000 C CNN
 F 1 "600S2R7" V 6389 3600 50  0000 C CNN
 F 2 "Capacitor_SMD:C_0603_1608Metric" H 6600 3700 50  0001 C CNN
@@
 P 4200 4050
 AR Path="/5F177657/5F1BFC4F" Ref="L?"  Part="1"
-AR Path="/5F20B396/5F216BC6/5F1BFC4F" Ref="L6"  Part="1"
-F 0 "L6" V 4246 4127 50  0000 L CNN
+AR Path="/5F20B396/5F216BC6/5F1BFC4F" Ref="L7"  Part="1"
+F 0 "L7" V 4246 4127 50  0000 L CNN
 F 1 "0603HP-3N6X" V 4155 4127 50  0000 L CNN
 F 2 "Inductor_SMD:L_0603_1608Metric" H 3950 4200 50  0001 C CNN
@@
 P 3400 4300
 AR Path="/5F177657/5F1DD62C" Ref="#PWR?"  Part="1"
-AR Path="/5F20B396/5F216BC6/5F1DD62C" Ref="#PWR023"  Part="1"
-F 0 "#PWR023" H 3400 4050 50  0001 C CNN
+AR Path="/5F20B396/5F216BC6/5F1DD62C" Ref="#PWR025"  Part="1"
+F 0 "#PWR025" H 3400 4050 50  0001 C CNN
 F 1 "GNDA" H 3405 4127 50  0000 C CNN
 F 2 "" H 3400 4300 50  0001 C CNN
@@
 P 5000 4300
 AR Path="/5F177657/5F1DEE33" Ref="#PWR?"  Part="1"
-AR Path="/5F20B396/5F216BC6/5F1DEE33" Ref="#PWR025"  Part="1"
-F 0 "#PWR025" H 5000 4050 50  0001 C CNN
+AR Path="/5F20B396/5F216BC6/5F1DEE33" Ref="#PWR027"  Part="1"
+F 0 "#PWR027" H 5000 4050 50  0001 C CNN
 F 1 "GNDA" H 5005 4127 50  0000 C CNN
 F 2 "" H 5000 4300 50  0001 C CNN
@@
 P 4200 4500
 AR Path="/5F177657/5F1DF153" Ref="#PWR?"  Part="1"
-AR Path="/5F20B396/5F216BC6/5F1DF153" Ref="#PWR024"  Part="1"
-F 0 "#PWR024" H 4200 4250 50  0001 C CNN
+AR Path="/5F20B396/5F216BC6/5F1DF153" Ref="#PWR026"  Part="1"
+F 0 "#PWR026" H 4200 4250 50  0001 C CNN
 F 1 "GNDA" H 4205 4327 50  0000 C CNN
 F 2 "" H 4200 4500 50  0001 C CNN
@@
 P 7700 4500
 AR Path="/5F177657/5F1E005D" Ref="#PWR?"  Part="1"
-AR Path="/5F20B396/5F216BC6/5F1E005D" Ref="#PWR027"  Part="1"
-F 0 "#PWR027" H 7700 4250 50  0001 C CNN
+AR Path="/5F20B396/5F216BC6/5F1E005D" Ref="#PWR029"  Part="1"
+F 0 "#PWR029" H 7700 4250 50  0001 C CNN
 F 1 "GNDA" H 7705 4327 50  0000 C CNN
 F 2 "" H 7700 4500 50  0001 C CNN
@@
 P 6900 4300
 AR Path="/5F177657/5F1E0461" Ref="#PWR?"  Part="1"
-AR Path="/5F20B396/5F216BC6/5F1E0461" Ref="#PWR026"  Part="1"
-F 0 "#PWR026" H 6900 4050 50  0001 C CNN
+AR Path="/5F20B396/5F216BC6/5F1E0461" Ref="#PWR028"  Part="1"
+F 0 "#PWR028" H 6900 4050 50  0001 C CNN
 F 1 "GNDA" H 6905 4127 50  0000 C CNN
 F 2 "" H 6900 4300 50  0001 C CNN
@@
 P 8500 4300
 AR Path="/5F177657/5F1E096E" Ref="#PWR?"  Part="1"
-AR Path="/5F20B396/5F216BC6/5F1E096E" Ref="#PWR028"  Part="1"
-F 0 "#PWR028" H 8500 4050 50  0001 C CNN
+AR Path="/5F20B396/5F216BC6/5F1E096E" Ref="#PWR030"  Part="1"
+F 0 "#PWR030" H 8500 4050 50  0001 C CNN
 F 1 "GNDA" H 8505 4127 50  0000 C CNN
 F 2 "" H 8500 4300 50  0001 C CNN
